Commit message: arm_utils:writing obstcle avodnc logic-py

File: src/amr_description/urdf/amr.urdf.xacro (robot description, xacro)
@@ -21,4 +21,5 @@
         <mesh filename="package://amr_description/meshes/base_link.STL" />
       </geometry>
+      <material name="blue">
     </visual>
     <collision>
